Commit message: redamed greifer stl file in gripper_macro.urdf.xacro

File: ws_dependencies/description_beerpong/urdf/gripper_macro.urdf.xacro (robot description, xacro)
@@ -40,5 +40,5 @@
         <origin xyz="0 0 0" rpy="0 0 0" />
         <geometry>
-          <mesh filename="package://description_beerpong/meshes/visual/greifer_beerpong_baugruppe.stl" scale="0.001 0.001 0.001"/>
+          <mesh filename="package://description_beerpong/meshes/visual/greifer_beerpong_baugruppe_aussen_greifen.stl" scale="0.001 0.001 0.001"/>
         </geometry>
         <material name="${tf_prefix}grey" />
@@ -47,5 +47,5 @@
         <origin xyz="0 0 0" rpy="0 0 0" />
         <geometry>
-          <mesh filename="package://description_beerpong/meshes/collision/greifer_beerpong_baugruppe.stl" scale="0.001 0.001 0.001"/>
+          <mesh filename="package://description_beerpong/meshes/collision/greifer_beerpong_baugruppe_aussen_greifen.stl" scale="0.001 0.001 0.001"/>
         </geometry>
         <material name="${tf_prefix}red" />

Commit message: adjusted tcp_link z position

File: ws_dependencies/description_beerpong/urdf/gripper_macro.urdf.xacro (robot description, xacro)
@@ -100,5 +100,5 @@
     <!--add a TCP Link for convenience, show TCP reference set in rviz-->
     <joint name="${tf_prefix}tcp_joint" type="fixed">
-        <origin xyz="0 0.139 0" rpy="1.57075 0 3.1415"/>
+        <origin xyz="0 0.112 0" rpy="1.57075 0 3.1415"/>
         <parent link="${tf_prefix}gripper_link"/>
         <child link="${tf_prefix}tcp_link"/>
