Commit message: added cup dispenser to urdf

File: ws_dependencies/description_beerpong/urdf/full_robot.urdf.xacro (robot description, xacro)
@@ -139,3 +139,24 @@
       </collision>
     </link>
+    <!--Cup dispenser-->
+    <joint name="neobotix_to_cup_dispenser" type="fixed">
+        <origin xyz="0 0 0" rpy="0 0 0" />
+        <parent link="base_neobotix_link"/>
+        <child link="cup_dispenser_link"/>
+    </joint>
+    <link name="cup_dispenser_link">
+      <visual>
+        <origin xyz="0 0 0" rpy="0 0 0" />
+        <geometry>
+          <mesh filename="package://description_beerpong/meshes/visual/becherspender.stl" scale="0.001 0.001 0.001"/>
+        </geometry>
+      </visual>
+      <collision>
+        <origin xyz="0 0 0" rpy="0 0 0" />
+        <geometry>
+          <mesh filename="package://description_beerpong/meshes/collision/becherspender.stl" scale="0.001 0.001 0.001"/>
+        </geometry>
+        <material name="$(arg tf_prefix)red" />
+      </collision>
+    </link>
 </robot>

Commit message: changed translation and rotation of cup_dispenser in urdf

File: ws_dependencies/description_beerpong/urdf/full_robot.urdf.xacro (robot description, xacro)
@@ -141,5 +141,5 @@
     <!--Cup dispenser-->
     <joint name="neobotix_to_cup_dispenser" type="fixed">
-        <origin xyz="0 0 0" rpy="0 0 0" />
+        <origin xyz="-0.11 0.256 1.434" rpy="3.1415 0 3.1415" />
         <parent link="base_neobotix_link"/>
         <child link="cup_dispenser_link"/>

Commit message: changed coloor and position of cup_dispenser

File: ws_dependencies/description_beerpong/urdf/full_robot.urdf.xacro (robot description, xacro)
@@ -141,5 +141,5 @@
     <!--Cup dispenser-->
     <joint name="neobotix_to_cup_dispenser" type="fixed">
-        <origin xyz="-0.11 0.256 1.434" rpy="3.1415 0 3.1415" />
+        <origin xyz="-0.115 0.256 1.433" rpy="3.1415 0 3.1415" />
         <parent link="base_neobotix_link"/>
         <child link="cup_dispenser_link"/>
@@ -151,4 +151,5 @@
           <mesh filename="package://description_beerpong/meshes/visual/becherspender.stl" scale="0.001 0.001 0.001"/>
         </geometry>
+        <material name="$(arg tf_prefix)grey" />
       </visual>
       <collision>

Commit message: change tf_prefix to prefix

File: ws_dependencies/description_beerpong/urdf/full_robot.urdf.xacro (robot description, xacro)
@@ -9,5 +9,5 @@
    <xacro:arg name="ur_type" default="ur5x"/>
    <!-- parameters -->
-   <xacro:arg name="tf_prefix" default="" />
+   <xacro:arg name="prefix" default="ur_" />
    <xacro:arg name="joint_limit_params" default="$(find ur_description)/config/$(arg ur_type)/joint_limits.yaml"/>
    <xacro:arg name="kinematics_params" default="$(find ur_description)/config/$(arg ur_type)/default_kinematics.yaml"/>
@@ -51,8 +51,8 @@
    <!-- create link fixed to the "world" -->
    <link name="world" />
-     <!-- arm, ur base_link = world, neobotix under world z = 0 (only for collision avioidance)      parent="base_neobotix_link"-->
+     <!-- arm, ur base_link = world, neobotix under world z = 0 (only for collision avioidance)      parent="base_link"-->
    <xacro:ur_robot
      name="$(arg name)"
-     tf_prefix="$(arg tf_prefix)"
+     tf_prefix="$(arg prefix)"
      parent="world"
      joint_limits_parameters_file="$(arg joint_limit_params)"
@@ -108,5 +108,5 @@
       <plugin filename="libign_ros2_control-system.so" name="ign_ros2_control::IgnitionROS2ControlPlugin">
         <parameters>$(arg simulation_controllers)</parameters>
-        <controller_manager_node_name>$(arg tf_prefix)controller_manager</controller_manager_node_name>
+        <controller_manager_node_name>$(arg prefix)controller_manager</controller_manager_node_name>
       </plugin>
     </gazebo>
@@ -114,5 +114,5 @@
     <!--Greifer + Kamerahalter + Kamera Macro importieren -->
     <xacro:include filename="$(find description_beerpong)/urdf/gripper_macro.urdf.xacro"/>
-    <xacro:gripper_camera tf_prefix="$(arg tf_prefix)" parent="tool0" origin_xyz="0 0 0" origin_rpy="0 0 3.1415"/>
+    <xacro:gripper_camera prefix="$(arg prefix)" parent="tool0" origin_xyz="0 0 0" origin_rpy="0 0 3.1415"/>
     <!--Neobotix Macro importieren -->
     <xacro:include filename="$(find neo_mpo_500-2)/robot_model/mpo_500_macro.urdf.xacro"/>
@@ -121,5 +121,5 @@
     <joint name="neobotix_to_cabin" type="fixed">
         <origin xyz="0.072 0 0.386" rpy="0 0 -1.57075" />
-        <parent link="base_neobotix_link"/>
+        <parent link="base_link"/>
         <child link="cabin_link"/>
     </joint>
@@ -136,5 +136,5 @@
           <mesh filename="package://description_beerpong/meshes/collision/cabin.dae" scale="0.001 0.001 0.001"/>
         </geometry>
-        <material name="$(arg tf_prefix)red" />
+        <material name="$(arg prefix)red" />
       </collision>
     </link>
@@ -142,5 +142,5 @@
     <joint name="neobotix_to_cup_dispenser" type="fixed">
         <origin xyz="-0.115 0.256 1.433" rpy="3.1415 0 3.1415" />
-        <parent link="base_neobotix_link"/>
+        <parent link="base_link"/>
         <child link="cup_dispenser_link"/>
     </joint>
@@ -151,5 +151,5 @@
           <mesh filename="package://description_beerpong/meshes/visual/becherspender.stl" scale="0.001 0.001 0.001"/>
         </geometry>
-        <material name="$(arg tf_prefix)grey" />
+        <material name="$(arg prefix)grey" />
       </visual>
       <collision>
@@ -158,5 +158,5 @@
           <mesh filename="package://description_beerpong/meshes/collision/becherspender.stl" scale="0.001 0.001 0.001"/>
         </geometry>
-        <material name="$(arg tf_prefix)red" />
+        <material name="$(arg prefix)red" />
       </collision>
     </link>

File: ws_dependencies/description_beerpong/urdf/gripper_macro.urdf.xacro (robot description, xacro)
@@ -4,13 +4,13 @@
   <xacro:include filename="$(find description_beerpong)/urdf/materials.urdf.xacro" />
 <!--build the gripper links and joints using a macro, which will be called in the diy_gripper_model.urdf.xacro while launching-->
-  <xacro:macro name="gripper_camera" params="tf_prefix parent origin_xyz origin_rpy">
-    <xacro:materials tf_prefix="${tf_prefix}"/>
-    <joint name="${tf_prefix}gripper_to_parent" type="fixed">
+  <xacro:macro name="gripper_camera" params="prefix parent origin_xyz origin_rpy">
+    <xacro:materials prefix="${prefix}"/>
+    <joint name="${prefix}gripper_to_parent" type="fixed">
         <parent link="${parent}"/>
-        <child link="${tf_prefix}camera_mount_link"/>
+        <child link="${prefix}camera_mount_link"/>
         <origin xyz="${origin_xyz}" rpy="${origin_rpy}"/>
     </joint>
 <!-- Camera Mount-->
-    <link name="${tf_prefix}camera_mount_link">
+    <link name="${prefix}camera_mount_link">
       <visual>
         <origin xyz="0 0 0" rpy="0 0 0" />
@@ -18,5 +18,5 @@
           <mesh filename="package://description_beerpong/meshes/visual/Kamera_Mount.stl" scale="0.001 0.001 0.001"/>
         </geometry>
-        <material name="${tf_prefix}grey" />
+        <material name="${prefix}grey" />
       </visual>
       <collision>
@@ -25,16 +25,16 @@
           <mesh filename="package://description_beerpong/meshes/collision/Kamera_Mount.stl" scale="0.001 0.001 0.001"/>
         </geometry>
-        <material name="${tf_prefix}red" />
+        <material name="${prefix}red" />
       </collision>
     </link>
 <!-- Gripper + Finger + Adapter-Plate-->
-    <joint name="${tf_prefix}gripper_joint" type="fixed">
+    <joint name="${prefix}gripper_joint" type="fixed">
     <!-- Position zueinander wird in den joints angepasst (nicht in links)-->
       <origin xyz="0 0 0.0245" rpy="1.57075 0 3.1415" />
-      <parent link="${tf_prefix}camera_mount_link" />
-      <child link="${tf_prefix}gripper_link" />
+      <parent link="${prefix}camera_mount_link" />
+      <child link="${prefix}gripper_link" />
       <axis xyz="0 0 1" />
     </joint>
-    <link name="${tf_prefix}gripper_link">
+    <link name="${prefix}gripper_link">
       <visual>
         <origin xyz="0 0 0" rpy="0 0 0" />
@@ -42,5 +42,5 @@
           <mesh filename="package://description_beerpong/meshes/visual/greifer_beerpong_baugruppe_aussen_greifen.stl" scale="0.001 0.001 0.001"/>
         </geometry>
-        <material name="${tf_prefix}grey" />
+        <material name="${prefix}grey" />
       </visual>
       <collision>
@@ -49,12 +49,12 @@
           <mesh filename="package://description_beerpong/meshes/collision/greifer_beerpong_baugruppe_aussen_greifen.stl" scale="0.001 0.001 0.001"/>
         </geometry>
-        <material name="${tf_prefix}red" />
+        <material name="${prefix}red" />
       </collision>
     </link>
 <!-- Realsense-Camera -->
-    <joint name="${tf_prefix}camera_joint" type="fixed">
+    <joint name="${prefix}camera_joint" type="fixed">
       <origin xyz="0 0.098 0.074" rpy="0 0 3.1415" />
-      <parent link="${tf_prefix}camera_mount_link" />
-      <child link="${tf_prefix}camera_link" />
+      <parent link="${prefix}camera_mount_link" />
+      <child link="${prefix}camera_link" />
       <axis xyz="0 0 1" />
     </joint>
@@ -66,5 +66,5 @@
       <origin xyz="0 0.098 0.074" rpy="0 0 0"/>
     </xacro:sensor_d415> -->
-    <link name="${tf_prefix}camera_link">
+    <link name="${prefix}camera_link">
       <visual>
         <origin xyz="0 0 0" rpy="0 0 0" />
@@ -72,5 +72,5 @@
           <mesh filename="package://description_beerpong/meshes/visual/realsense415.stl" scale="1 1 1"/>
         </geometry>
-        <material name="${tf_prefix}grey" />
+        <material name="${prefix}grey" />
       </visual>
       <collision>
@@ -79,8 +79,8 @@
           <mesh filename="package://description_beerpong/meshes/collision/realsense415.stl" scale="1 1 1"/>
         </geometry>
-        <material name="${tf_prefix}red" />
+        <material name="${prefix}red" />
       </collision>
     </link>
-    <!-- <link name="${tf_prefix}camera_link">
+    <!-- <link name="${prefix}camera_link">
       <visual>
         <origin xyz="0 0 0" rpy="0 0 0" />
@@ -88,5 +88,5 @@
           <mesh filename="package://description_beerpong/meshes/visual/realsense415.stl" scale="1 1 1"/>
         </geometry>
-        <material name="${tf_prefix}grey" />
+        <material name="${prefix}grey" />
       </visual>
       <collision>
@@ -95,14 +95,14 @@
           <mesh filename="package://description_beerpong/meshes/collision/realsense415.stl"  scale="1 1 1"/>
         </geometry>
-        <material name="${tf_prefix}red" />
+        <material name="${prefix}red" />
       </collision>
     </link> -->
     <!--add a TCP Link for convenience, show TCP reference set in rviz-->
-    <joint name="${tf_prefix}tcp_joint" type="fixed">
+    <joint name="${prefix}tcp_joint" type="fixed">
         <origin xyz="0 0.112 0" rpy="1.57075 0 3.1415"/>
-        <parent link="${tf_prefix}gripper_link"/>
-        <child link="${tf_prefix}tcp_link"/>
+        <parent link="${prefix}gripper_link"/>
+        <child link="${prefix}tcp_link"/>
     </joint>
-    <link name="${tf_prefix}tcp_link"/>
+    <link name="${prefix}tcp_link"/>
   </xacro:macro>
 </robot>

File: ws_dependencies/description_beerpong/urdf/materials.urdf.xacro (robot description, xacro)
@@ -5,30 +5,30 @@
 -->
 <robot xmlns:xacro="http://wiki.ros.org/xacro">
-  <xacro:macro name="materials" params="tf_prefix">
-    <material name="${tf_prefix}black">
+  <xacro:macro name="materials" params="prefix">
+    <material name="${prefix}black">
       <color rgba="0.0 0.0 0.0 1.0"/>
     </material>
-    <material name="${tf_prefix}blue">
+    <material name="${prefix}blue">
       <color rgba="0.0 0.0 0.8 1.0"/>
     </material>
-    <material name="${tf_prefix}green">
+    <material name="${prefix}green">
       <color rgba="0.0 0.8 0.0 1.0"/>
     </material>
-    <material name="${tf_prefix}yellow">
+    <material name="${prefix}yellow">
       <color rgba="1.0 1.0 0.0 1.0"/>
     </material>
-    <material name="${tf_prefix}grey">
+    <material name="${prefix}grey">
       <color rgba="0.6 0.6 0.6 1.0"/>
     </material>
-    <material name="${tf_prefix}orange">
+    <material name="${prefix}orange">
       <color rgba="${255/255} ${108/255} ${10/255} 1.0"/>
     </material>
-    <material name="${tf_prefix}brown">
+    <material name="${prefix}brown">
       <color rgba="${222/255} ${207/255} ${195/255} 1.0"/>
     </material>
-    <material name="${tf_prefix}red">
+    <material name="${prefix}red">
       <color rgba="0.8 0.0 0.0 1.0"/>
     </material>
-    <material name="${tf_prefix}white">
+    <material name="${prefix}white">
       <color rgba="1.0 1.0 1.0 1.0"/>
     </material>

Commit message: switch back to full urdf nbtx+ur

File: ws_dependencies/description_beerpong/urdf/full_robot.urdf.xacro (robot description, xacro)
@@ -116,8 +116,8 @@
     <xacro:gripper_camera tf_prefix="$(arg tf_prefix)" parent="$(arg tf_prefix)tool0" origin_xyz="0 0 0" origin_rpy="0 0 3.1415"/>
     <!--Neobotix Macro importieren -->
-    <!-- <xacro:include filename="$(find neo_mpo_500-2)/robot_model/mpo_500_macro.urdf.xacro"/>
-    <xacro:neobotix parent="world" origin_xyz="0 -0.205 -0.805" origin_rpy="0 0 1.57075"/> -->
+    <xacro:include filename="$(find neo_mpo_500-2)/robot_model/mpo_500_macro.urdf.xacro"/>
+    <xacro:neobotix parent="world" origin_xyz="0 -0.205 -0.805" origin_rpy="0 0 1.57075"/>
     <!--Neobotix cabin-->
-    <!-- <joint name="neobotix_to_cabin" type="fixed">
+    <joint name="neobotix_to_cabin" type="fixed">
         <origin xyz="0.072 0 0.386" rpy="0 0 -1.57075" />
         <parent link="base_link"/>
@@ -138,8 +138,8 @@
         <material name="$(arg tf_prefix)red" />
       </collision>
-    </link> -->
+    </link>
     <!--Cup dispenser-->
     <joint name="neobotix_to_cup_dispenser" type="fixed">
-        <!-- <origin xyz="-0.115 0.256 1.433" rpy="3.1415 0 3.1415" /> -->
+        <!-- <origin xyz="-0.115 0.256 1.433" rpy="3.1415 0 3.1415" /> to nbtx base_link -->
         <origin xyz="-0.256 -0.33 0.635" rpy="3.1415 0 -1.57075" />
         <parent link="world"/>

Commit message: add new description package version (equals the one in the neo_mpo_500 bringup repo)

File: ws_dependencies/description_beerpong/urdf/full_robot.urdf.xacro (robot description, xacro)
@@ -50,10 +50,36 @@
    <xacro:property name="initial_positions_file" default="$(arg initial_positions_file)"/>
    <!-- create link fixed to the "world" -->
-   <link name="world" />
+   <!--<link name="world" />-->
+    <!--Neobotix Macro importieren -->
+    <xacro:include filename="$(find neo_mpo_500-2)/robot_model/mpo_500_macro.urdf.xacro"/>
+    <xacro:neobotix/>
+    <!--<xacro:neobotix parent="world" origin_xyz="0 -0.205 -0.805" origin_rpy="0 0 1.57075"/>-->
+    <!--Neobotix cabin-->
+    <joint name="neobotix_to_cabin" type="fixed">
+        <origin xyz="0.072 0 0.386" rpy="0 0 -1.57075" />
+        <parent link="base_link"/>
+        <child link="cabin_link"/>
+    </joint>
+    <link name="cabin_link">
+      <visual>
+        <origin xyz="0 0 0" rpy="0 0 0" />
+        <geometry>
+          <mesh filename="package://description_beerpong/meshes/visual/cabin.dae" scale="0.001 0.001 0.001"/>
+        </geometry>
+      </visual>
+      <collision>
+        <origin xyz="0 0 0" rpy="0 0 0" />
+        <geometry>
+          <mesh filename="package://description_beerpong/meshes/collision/cabin.dae" scale="0.001 0.001 0.001"/>
+        </geometry>
+        <material name="$(arg tf_prefix)red" />
+      </collision>
+    </link>
      <!-- arm, ur base_link = world, neobotix under world z = 0 (only for collision avioidance)      parent="base_link"-->
+     <!-- neobotix base link is parent -->
    <xacro:ur_robot
      name="$(arg name)"
      tf_prefix="$(arg tf_prefix)"
-     parent="world"
+     parent="base_link"
      joint_limits_parameters_file="$(arg joint_limit_params)"
      kinematics_parameters_file="$(arg kinematics_params)"
@@ -89,8 +115,9 @@
      trajectory_port="$(arg trajectory_port)"
      >
-     <origin xyz="0 0 0" rpy="0 0 0"/>         <!-- position robot in the world origin xyz="0.205 0 0.805" rpy="0 0 -1.57075"-->
+     <origin xyz="0.205 0 0.805" rpy="0 0 -1.57075"/>         <!-- position robot in the world origin xyz="0.205 0 0.805" rpy="0 0 -1.57075"-->
    </xacro:ur_robot>
-  <xacro:if value="$(arg sim_gazebo)">
-    <!-- Gazebo plugins -->
+  <!-- NEVER USED -->
+  <!-- <xacro:if value="$(arg sim_gazebo)">
+    < Gazebo plugins>
     <gazebo reference="world">
     </gazebo>
@@ -102,5 +129,5 @@
   </xacro:if>
   <xacro:if value="$(arg sim_ignition)">
-    <!-- Gazebo plugins -->
+    <!Gazebo plugins>
     <gazebo reference="world">
     </gazebo>
@@ -111,37 +138,13 @@
       </plugin>
     </gazebo>
-  </xacro:if>
+  </xacro:if> -->
     <!--Greifer + Kamerahalter + Kamera Macro importieren -->
     <xacro:include filename="$(find description_beerpong)/urdf/gripper_macro.urdf.xacro"/>
     <xacro:gripper_camera tf_prefix="$(arg tf_prefix)" parent="$(arg tf_prefix)tool0" origin_xyz="0 0 0" origin_rpy="0 0 3.1415"/>
-    <!--Neobotix Macro importieren -->
-    <xacro:include filename="$(find neo_mpo_500-2)/robot_model/mpo_500_macro.urdf.xacro"/>
-    <xacro:neobotix parent="world" origin_xyz="0 -0.205 -0.805" origin_rpy="0 0 1.57075"/>
-    <!--Neobotix cabin-->
-    <joint name="neobotix_to_cabin" type="fixed">
-        <origin xyz="0.072 0 0.386" rpy="0 0 -1.57075" />
-        <parent link="base_link"/>
-        <child link="cabin_link"/>
-    </joint>
-    <link name="cabin_link">
-      <visual>
-        <origin xyz="0 0 0" rpy="0 0 0" />
-        <geometry>
-          <mesh filename="package://description_beerpong/meshes/visual/cabin.dae" scale="0.001 0.001 0.001"/>
-        </geometry>
-      </visual>
-      <collision>
-        <origin xyz="0 0 0" rpy="0 0 0" />
-        <geometry>
-          <mesh filename="package://description_beerpong/meshes/collision/cabin.dae" scale="0.001 0.001 0.001"/>
-        </geometry>
-        <material name="$(arg tf_prefix)red" />
-      </collision>
-    </link>
     <!--Cup dispenser-->
     <joint name="neobotix_to_cup_dispenser" type="fixed">
-        <!-- <origin xyz="-0.115 0.256 1.433" rpy="3.1415 0 3.1415" /> to nbtx base_link -->
-        <origin xyz="-0.256 -0.33 0.635" rpy="3.1415 0 -1.57075" />
-        <parent link="world"/>
+        <origin xyz="-0.115 0.256 1.433" rpy="3.1415 0 3.1415" />
+        <!-- <origin xyz="-0.256 -0.33 0.635" rpy="3.1415 0 -1.57075" />  world to cup dispenser -->
+        <parent link="base_link"/>
         <child link="cup_dispenser_link"/>
     </joint>
@@ -165,10 +168,10 @@
     <joint name="ur_to_collision_plane" type="fixed">
         <origin xyz="0.0 0.0 0.0" rpy="0.0 0.0 0.0" />
-        <parent link="world"/>
+        <parent link="base_link"/>
         <child link="collision_plane_link"/>
     </joint>
     <link name="collision_plane_link">
       <collision>
-        <origin xyz="0 0 -0.02" rpy="0 0 0" />
+        <origin xyz="0 0 0.803" rpy="0 0 0" />
         <geometry>
           <cylinder radius="1.0" length="0.02"/>
@@ -176,11 +179,4 @@
         <material name="$(arg tf_prefix)red" />
       </collision>
-      <visual>
-        <origin xyz="0 0 -0.02" rpy="0 0 0" />
-        <geometry>
-          <cylinder radius="1.0" length="0.02"/>
-        </geometry>
-        <material name="$(arg tf_prefix)grey" />
-      </visual>
     </link>
 </robot>

Commit message: add world link to urdf

File: ws_dependencies/description_beerpong/urdf/full_robot.urdf.xacro (robot description, xacro)
@@ -76,4 +76,11 @@
       </collision>
     </link>
+    <!--world link for convenience-->
+    <link name="world"/>
+     <joint name="neobotix_to_world" type="fixed">
+        <origin xyz="0.205 0 0.805" rpy="0 0 -1.57075"/>
+        <parent link="base_link"/>
+        <child link="world"/>
+    </joint>
      <!-- arm, ur base_link = world, neobotix under world z = 0 (only for collision avioidance)      parent="base_link"-->
      <!-- neobotix base link is parent -->
@@ -81,5 +88,5 @@
      name="$(arg name)"
      tf_prefix="$(arg tf_prefix)"
-     parent="base_link"
+     parent="world"
      joint_limits_parameters_file="$(arg joint_limit_params)"
      kinematics_parameters_file="$(arg kinematics_params)"
@@ -115,5 +122,5 @@
      trajectory_port="$(arg trajectory_port)"
      >
-     <origin xyz="0.205 0 0.805" rpy="0 0 -1.57075"/>         <!-- position robot in the world origin xyz="0.205 0 0.805" rpy="0 0 -1.57075"-->
+     <origin xyz="0 0 0" rpy="0 0 0"/>         <!-- position robot in the world origin xyz="0.205 0 0.805" rpy="0 0 -1.57075"-->
    </xacro:ur_robot>
   <!-- NEVER USED -->
