Commit message: second branch for testing purposes - 2 robot state publishers, this without nbtx

File: ws_dependencies/description_beerpong/urdf/full_robot.urdf.xacro (robot description, xacro)
@@ -49,12 +49,10 @@
    <!-- convert to property to use substitution in function -->
    <xacro:property name="initial_positions_file" default="$(arg initial_positions_file)"/>
-   <!-- create link fixed to the "world" -->
-   <!--<link name="world" />-->
     <!--Neobotix Macro importieren -->
-    <xacro:include filename="$(find neo_mpo_500-2)/robot_model/mpo_500_macro.urdf.xacro"/>
-    <xacro:neobotix/>
+    <!-- <xacro:include filename="$(find neo_mpo_500-2)/robot_model/mpo_500_macro.urdf.xacro"/>
+    <xacro:neobotix/> -->
     <!--<xacro:neobotix parent="world" origin_xyz="0 -0.205 -0.805" origin_rpy="0 0 1.57075"/>-->
     <!--Neobotix cabin-->
-    <joint name="neobotix_to_cabin" type="fixed">
+    <!-- <joint name="neobotix_to_cabin" type="fixed">
         <origin xyz="0.072 0 0.386" rpy="0 0 -1.57075" />
         <parent link="base_link"/>
@@ -75,12 +73,12 @@
         <material name="$(arg tf_prefix)red" />
       </collision>
-    </link>
+    </link> -->
     <!--world link for convenience-->
     <link name="world"/>
-     <joint name="neobotix_to_world" type="fixed">
+     <!-- <joint name="neobotix_to_world" type="fixed">
         <origin xyz="0.205 0 0.805" rpy="0 0 -1.57075"/>
         <parent link="base_link"/>
         <child link="world"/>
-    </joint>
+    </joint>  -->
      <!-- arm, ur base_link = world, neobotix under world z = 0 (only for collision avioidance)      parent="base_link"-->
      <!-- neobotix base link is parent -->
@@ -151,7 +149,7 @@
     <!--Cup dispenser-->
     <joint name="neobotix_to_cup_dispenser" type="fixed">
-        <origin xyz="-0.115 0.256 1.433" rpy="3.1415 0 3.1415" />
-        <!-- <origin xyz="-0.256 -0.33 0.635" rpy="3.1415 0 -1.57075" />  world to cup dispenser -->
-        <parent link="base_link"/>
+        <!-- <origin xyz="-0.115 0.256 1.433" rpy="3.1415 0 3.1415" /> -->
+        <origin xyz="-0.256 -0.33 0.635" rpy="3.1415 0 -1.57075" />  <!--world to cup dispenser-->
+        <parent link="world"/>
         <child link="cup_dispenser_link"/>
     </joint>
@@ -175,10 +173,10 @@
     <joint name="ur_to_collision_plane" type="fixed">
         <origin xyz="0.0 0.0 0.0" rpy="0.0 0.0 0.0" />
-        <parent link="base_link"/>
+        <parent link="world"/>
         <child link="collision_plane_link"/>
     </joint>
     <link name="collision_plane_link">
       <collision>
-        <origin xyz="0 0 0.803" rpy="0 0 0" />
+        <origin xyz="0 0 0.03" rpy="0 0 0" />
         <geometry>
           <cylinder radius="1.0" length="0.02"/>
