Commit message: change base_neobotix_link to base_link

File: ws_dependencies/neo_mpo_500-2-humble/robot_model/mpo_500_macro.urdf.xacro (robot description, xacro)
@@ -4,14 +4,14 @@
       <joint name="neobotix_to_parent" type="fixed">
           <parent link="${parent}"/>
-          <child link="base_neobotix_link"/>
+          <child link="base_link"/>
           <origin xyz="${origin_xyz}" rpy="${origin_rpy}"/>
       </joint>
       <!-- Base Macro-->
-      <link name="base_neobotix_link"/>
+      <link name="base_link"/>
       <joint name="base_footprint_joint" type="fixed">
         <origin rpy="0 0 0" xyz="0 0 0"/>
         <axis xyz="0 0 -1"/>
         <joint_properties damping="1" friction="1"/>
-        <parent link="base_neobotix_link"/>
+        <parent link="base_link"/>
         <child link="base_footprint"/>
       </joint>
@@ -152,5 +152,5 @@
         <axis xyz="0 1 0"/>
         <origin rpy="0 0 0" xyz="0.442 0 0.372"/>
-        <parent link="base_neobotix_link"/>
+        <parent link="base_link"/>
         <child link="lidar_1_link"/>
       </joint>
@@ -177,5 +177,5 @@
         <axis xyz="0 1 0"/>
         <origin rpy="0 0 3.14" xyz="-0.442 0 0.372"/>
-        <parent link="base_neobotix_link"/>
+        <parent link="base_link"/>
         <child link="lidar_2_link"/>
       </joint>
