Commit message: add prefix to ur

File: ws_dependencies/beerpong_moveit_config/srdf/beerpong_macro.srdf.xacro (robot description, xacro)
@@ -5,5 +5,5 @@
     A URDF file must exist for this robot as well, where the joints and the links that are referenced are defined
 -->
-  <xacro:macro name="ur_srdf" params="name prefix">
+  <xacro:macro name="ur_srdf" params="name tf_prefix">
     <!--GROUPS - Representation of a set of joints and links. This can be useful for specifying DOF to plan for, defining arms, end effectors, etc-->
     <!--LINKS - When a link is specified, the parent joint of that link (if it exists) is automatically included-->
@@ -12,32 +12,32 @@
     <!--SUBGROUPS - Groups can also be formed by referencing to already defined group names-->
     <!--define start and end of the kinematic chain-->
-    <group name="${prefix}${name}_manipulator">
-      <chain base_link="${prefix}base_link" tip_link="${prefix}tcp_link" />
-      <!--<chain base_link="${prefix}base_link" tip_link="${prefix}camera_link" />-->
+    <group name="${name}_manipulator">
+      <chain base_link="${tf_prefix}base_link" tip_link="${tf_prefix}tcp_link" />
+      <!--<chain base_link="${tf_prefix}base_link" tip_link="${tf_prefix}camera_link" />-->
     </group>
     <!--GROUP STATES - Purpose - Define a named state for a particular group, in terms of joint values. This is useful to define states like 'folded arms'-->
-    <group_state name="${prefix}home" group="${prefix}${name}_manipulator">
-      <joint name="${prefix}elbow_joint" value="0" />
-      <joint name="${prefix}shoulder_lift_joint" value="-1.5707" />
-      <joint name="${prefix}shoulder_pan_joint" value="0" />
-      <joint name="${prefix}wrist_1_joint" value="0" />
-      <joint name="${prefix}wrist_2_joint" value="0" />
-      <joint name="${prefix}wrist_3_joint" value="0" />
+    <group_state name="${tf_prefix}home" group="${name}_manipulator">
+      <joint name="${tf_prefix}elbow_joint" value="0" />
+      <joint name="${tf_prefix}shoulder_lift_joint" value="-1.5707" />
+      <joint name="${tf_prefix}shoulder_pan_joint" value="0" />
+      <joint name="${tf_prefix}wrist_1_joint" value="0" />
+      <joint name="${tf_prefix}wrist_2_joint" value="0" />
+      <joint name="${tf_prefix}wrist_3_joint" value="0" />
     </group_state>
-    <group_state name="${prefix}up" group="${prefix}${name}_manipulator">
-      <joint name="${prefix}elbow_joint" value="0" />
-      <joint name="${prefix}shoulder_lift_joint" value="-1.5707" />
-      <joint name="${prefix}shoulder_pan_joint" value="0" />
-      <joint name="${prefix}wrist_1_joint" value="-1.5707" />
-      <joint name="${prefix}wrist_2_joint" value="0" />
-      <joint name="${prefix}wrist_3_joint" value="0" />
+    <group_state name="${tf_prefix}up" group="${tf_prefix}${name}_manipulator">
+      <joint name="${tf_prefix}elbow_joint" value="0" />
+      <joint name="${tf_prefix}shoulder_lift_joint" value="-1.5707" />
+      <joint name="${tf_prefix}shoulder_pan_joint" value="0" />
+      <joint name="${tf_prefix}wrist_1_joint" value="-1.5707" />
+      <joint name="${tf_prefix}wrist_2_joint" value="0" />
+      <joint name="${tf_prefix}wrist_3_joint" value="0" />
     </group_state>
-    <group_state name="${prefix}test_configuration" group="${prefix}${name}_manipulator">
-      <joint name="${prefix}elbow_joint" value="1.4" />
-      <joint name="${prefix}shoulder_lift_joint" value="-1.62" />
-      <joint name="${prefix}shoulder_pan_joint" value="1.54" />
-      <joint name="${prefix}wrist_1_joint" value="-1.2" />
-      <joint name="${prefix}wrist_2_joint" value="-1.6" />
-      <joint name="${prefix}wrist_3_joint" value="-0.11" />
+    <group_state name="${tf_prefix}test_configuration" group="${tf_prefix}${name}_manipulator">
+      <joint name="${tf_prefix}elbow_joint" value="1.4" />
+      <joint name="${tf_prefix}shoulder_lift_joint" value="-1.62" />
+      <joint name="${tf_prefix}shoulder_pan_joint" value="1.54" />
+      <joint name="${tf_prefix}wrist_1_joint" value="-1.2" />
+      <joint name="${tf_prefix}wrist_2_joint" value="-1.6" />
+      <joint name="${tf_prefix}wrist_3_joint" value="-0.11" />
     </group_state>
     <!--END EFFECTOR - Purpose - Represent information about an end effector.-->
@@ -53,22 +53,22 @@
     <disable_collisions link1="base_footprint" link2="lidar_2_link" reason="Adjacent" />
     <disable_collisions link1="base_footprint" link2="cabin_link" reason="Adjacent" />
-    <disable_collisions link1="cabin_link" link2="${prefix}base_link_inertia" reason="Adjacent" />
-    <disable_collisions link1="${prefix}base_link" link2="${prefix}base_link_inertia" reason="Adjacent" />
-    <disable_collisions link1="${prefix}base_link_inertia" link2="${prefix}shoulder_link" reason="Adjacent" />
-    <disable_collisions link1="${prefix}tool0" link2="${prefix}wrist_1_link" reason="Never" />
-    <disable_collisions link1="${prefix}tool0" link2="${prefix}wrist_2_link" reason="Never" />
-    <disable_collisions link1="${prefix}tool0" link2="${prefix}wrist_3_link" reason="Adjacent" />
-    <disable_collisions link1="${prefix}forearm_link" link2="${prefix}upper_arm_link" reason="Adjacent" />
-    <disable_collisions link1="${prefix}forearm_link" link2="${prefix}wrist_1_link" reason="Adjacent" />
-    <disable_collisions link1="${prefix}shoulder_link" link2="${prefix}upper_arm_link" reason="Adjacent" />
-    <disable_collisions link1="${prefix}wrist_1_link" link2="${prefix}wrist_2_link" reason="Adjacent" />
-    <disable_collisions link1="${prefix}wrist_1_link" link2="${prefix}wrist_3_link" reason="Never" />
-    <disable_collisions link1="${prefix}wrist_2_link" link2="${prefix}wrist_3_link" reason="Adjacent" />
+    <disable_collisions link1="cabin_link" link2="${tf_prefix}base_link_inertia" reason="Adjacent" />
+    <disable_collisions link1="${tf_prefix}base_link" link2="${tf_prefix}base_link_inertia" reason="Adjacent" />
+    <disable_collisions link1="${tf_prefix}base_link_inertia" link2="${tf_prefix}shoulder_link" reason="Adjacent" />
+    <disable_collisions link1="${tf_prefix}tool0" link2="${tf_prefix}wrist_1_link" reason="Never" />
+    <disable_collisions link1="${tf_prefix}tool0" link2="${tf_prefix}wrist_2_link" reason="Never" />
+    <disable_collisions link1="${tf_prefix}tool0" link2="${tf_prefix}wrist_3_link" reason="Adjacent" />
+    <disable_collisions link1="${tf_prefix}forearm_link" link2="${tf_prefix}upper_arm_link" reason="Adjacent" />
+    <disable_collisions link1="${tf_prefix}forearm_link" link2="${tf_prefix}wrist_1_link" reason="Adjacent" />
+    <disable_collisions link1="${tf_prefix}shoulder_link" link2="${tf_prefix}upper_arm_link" reason="Adjacent" />
+    <disable_collisions link1="${tf_prefix}wrist_1_link" link2="${tf_prefix}wrist_2_link" reason="Adjacent" />
+    <disable_collisions link1="${tf_prefix}wrist_1_link" link2="${tf_prefix}wrist_3_link" reason="Never" />
+    <disable_collisions link1="${tf_prefix}wrist_2_link" link2="${tf_prefix}wrist_3_link" reason="Adjacent" />
     <!--disable gripper and camera collisions-->
-    <disable_collisions link1="${prefix}wrist_3_link" link2="${prefix}camera_mount_link" reason="Adjacent" />
-    <disable_collisions link1="${prefix}camera_mount_link" link2="${prefix}gripper_link" reason="Adjacent" />
-    <disable_collisions link1="${prefix}camera_mount_link" link2="${prefix}camera_link" reason="Never" />
+    <disable_collisions link1="${tf_prefix}wrist_3_link" link2="${tf_prefix}camera_mount_link" reason="Adjacent" />
+    <disable_collisions link1="${tf_prefix}camera_mount_link" link2="${tf_prefix}gripper_link" reason="Adjacent" />
+    <disable_collisions link1="${tf_prefix}camera_mount_link" link2="${tf_prefix}camera_link" reason="Never" />
     <!--disable cabin and cup_dispeser collisions-->
-    <disable_collisions link1="${prefix}cabin_link" link2="${prefix}cup_dispenser_link" reason="Adjacent" />
+    <disable_collisions link1="cabin_link" link2="cup_dispenser_link" reason="Adjacent" />
   </xacro:macro>
 </robot>

File: ws_dependencies/beerpong_moveit_config/srdf/ur.srdf.xacro (robot description, xacro)
@@ -4,6 +4,6 @@
   <xacro:arg name="name" default="ur"/>
   <!-- parameters -->
-  <xacro:arg name="prefix" default="" />
+  <xacro:arg name="tf_prefix" default="" />
   <xacro:include filename="$(find beerpong_moveit_config)/srdf/beerpong_macro.srdf.xacro"/>
-  <xacro:ur_srdf name="$(arg name)" prefix="$(arg prefix)"/>
+  <xacro:ur_srdf name="$(arg name)" tf_prefix="$(arg tf_prefix)"/>
 </robot>

File: ws_dependencies/beerpong_moveit_config/srdf/ur_macro.srdf.xacro (robot description, xacro)
@@ -5,5 +5,5 @@
     A URDF file must exist for this robot as well, where the joints and the links that are referenced are defined
 -->
-  <xacro:macro name="ur_srdf" params="name prefix">
+  <xacro:macro name="ur_srdf" params="name tf_prefix">
     <!--GROUPS - Representation of a set of joints and links. This can be useful for specifying DOF to plan for, defining arms, end effectors, etc-->
     <!--LINKS - When a link is specified, the parent joint of that link (if it exists) is automatically included-->
@@ -11,46 +11,46 @@
     <!--CHAINS - When a chain is specified, all the links along the chain (including endpoints) are included in the group. Additionally, all the joints that are parents to included links are also included. This means that joints along the chain and the parent joint of the base link are included in the group-->
     <!--SUBGROUPS - Groups can also be formed by referencing to already defined group names-->
-    <group name="${prefix}${name}_manipulator">
-      <chain base_link="${prefix}base_link" tip_link="${prefix}tool0" />
+    <group name="${tf_prefix}${name}_manipulator">
+      <chain base_link="${tf_prefix}base_link" tip_link="${tf_prefix}tool0" />
     </group>
     <!--GROUP STATES - Purpose - Define a named state for a particular group, in terms of joint values. This is useful to define states like 'folded arms'-->
-    <group_state name="${prefix}home" group="${prefix}${name}_manipulator">
-      <joint name="${prefix}elbow_joint" value="0" />
-      <joint name="${prefix}shoulder_lift_joint" value="-1.5707" />
-      <joint name="${prefix}shoulder_pan_joint" value="0" />
-      <joint name="${prefix}wrist_1_joint" value="0" />
-      <joint name="${prefix}wrist_2_joint" value="0" />
-      <joint name="${prefix}wrist_3_joint" value="0" />
+    <group_state name="${tf_prefix}home" group="${tf_prefix}${name}_manipulator">
+      <joint name="${tf_prefix}elbow_joint" value="0" />
+      <joint name="${tf_prefix}shoulder_lift_joint" value="-1.5707" />
+      <joint name="${tf_prefix}shoulder_pan_joint" value="0" />
+      <joint name="${tf_prefix}wrist_1_joint" value="0" />
+      <joint name="${tf_prefix}wrist_2_joint" value="0" />
+      <joint name="${tf_prefix}wrist_3_joint" value="0" />
     </group_state>
-    <group_state name="${prefix}up" group="${prefix}${name}_manipulator">
-      <joint name="${prefix}elbow_joint" value="0" />
-      <joint name="${prefix}shoulder_lift_joint" value="-1.5707" />
-      <joint name="${prefix}shoulder_pan_joint" value="0" />
-      <joint name="${prefix}wrist_1_joint" value="-1.5707" />
-      <joint name="${prefix}wrist_2_joint" value="0" />
-      <joint name="${prefix}wrist_3_joint" value="0" />
+    <group_state name="${tf_prefix}up" group="${tf_prefix}${name}_manipulator">
+      <joint name="${tf_prefix}elbow_joint" value="0" />
+      <joint name="${tf_prefix}shoulder_lift_joint" value="-1.5707" />
+      <joint name="${tf_prefix}shoulder_pan_joint" value="0" />
+      <joint name="${tf_prefix}wrist_1_joint" value="-1.5707" />
+      <joint name="${tf_prefix}wrist_2_joint" value="0" />
+      <joint name="${tf_prefix}wrist_3_joint" value="0" />
     </group_state>
-    <group_state name="${prefix}test_configuration" group="${prefix}${name}_manipulator">
-      <joint name="${prefix}elbow_joint" value="1.4" />
-      <joint name="${prefix}shoulder_lift_joint" value="-1.62" />
-      <joint name="${prefix}shoulder_pan_joint" value="1.54" />
-      <joint name="${prefix}wrist_1_joint" value="-1.2" />
-      <joint name="${prefix}wrist_2_joint" value="-1.6" />
-      <joint name="${prefix}wrist_3_joint" value="-0.11" />
+    <group_state name="${tf_prefix}test_configuration" group="${tf_prefix}${name}_manipulator">
+      <joint name="${tf_prefix}elbow_joint" value="1.4" />
+      <joint name="${tf_prefix}shoulder_lift_joint" value="-1.62" />
+      <joint name="${tf_prefix}shoulder_pan_joint" value="1.54" />
+      <joint name="${tf_prefix}wrist_1_joint" value="-1.2" />
+      <joint name="${tf_prefix}wrist_2_joint" value="-1.6" />
+      <joint name="${tf_prefix}wrist_3_joint" value="-0.11" />
     </group_state>
     <!--END EFFECTOR - Purpose - Represent information about an end effector.-->
     <!--VIRTUAL JOINT - Purpose - this element defines a virtual joint between a robot link and an external frame of reference (considered fixed with respect to the robot)-->
     <!--DISABLE COLLISIONS - By default it is assumed that any link of the robot could potentially come into collision with any other link in the robot. This tag disables collision checking between a specified pair of links. -->
-    <disable_collisions link1="${prefix}base_link" link2="${prefix}base_link_inertia" reason="Adjacent" />
-    <disable_collisions link1="${prefix}base_link_inertia" link2="${prefix}shoulder_link" reason="Adjacent" />
-    <disable_collisions link1="${prefix}tool0" link2="${prefix}wrist_1_link" reason="Never" />
-    <disable_collisions link1="${prefix}tool0" link2="${prefix}wrist_2_link" reason="Never" />
-    <disable_collisions link1="${prefix}tool0" link2="${prefix}wrist_3_link" reason="Adjacent" />
-    <disable_collisions link1="${prefix}forearm_link" link2="${prefix}upper_arm_link" reason="Adjacent" />
-    <disable_collisions link1="${prefix}forearm_link" link2="${prefix}wrist_1_link" reason="Adjacent" />
-    <disable_collisions link1="${prefix}shoulder_link" link2="${prefix}upper_arm_link" reason="Adjacent" />
-    <disable_collisions link1="${prefix}wrist_1_link" link2="${prefix}wrist_2_link" reason="Adjacent" />
-    <disable_collisions link1="${prefix}wrist_1_link" link2="${prefix}wrist_3_link" reason="Never" />
-    <disable_collisions link1="${prefix}wrist_2_link" link2="${prefix}wrist_3_link" reason="Adjacent" />
+    <disable_collisions link1="${tf_prefix}base_link" link2="${tf_prefix}base_link_inertia" reason="Adjacent" />
+    <disable_collisions link1="${tf_prefix}base_link_inertia" link2="${tf_prefix}shoulder_link" reason="Adjacent" />
+    <disable_collisions link1="${tf_prefix}tool0" link2="${tf_prefix}wrist_1_link" reason="Never" />
+    <disable_collisions link1="${tf_prefix}tool0" link2="${tf_prefix}wrist_2_link" reason="Never" />
+    <disable_collisions link1="${tf_prefix}tool0" link2="${tf_prefix}wrist_3_link" reason="Adjacent" />
+    <disable_collisions link1="${tf_prefix}forearm_link" link2="${tf_prefix}upper_arm_link" reason="Adjacent" />
+    <disable_collisions link1="${tf_prefix}forearm_link" link2="${tf_prefix}wrist_1_link" reason="Adjacent" />
+    <disable_collisions link1="${tf_prefix}shoulder_link" link2="${tf_prefix}upper_arm_link" reason="Adjacent" />
+    <disable_collisions link1="${tf_prefix}wrist_1_link" link2="${tf_prefix}wrist_2_link" reason="Adjacent" />
+    <disable_collisions link1="${tf_prefix}wrist_1_link" link2="${tf_prefix}wrist_3_link" reason="Never" />
+    <disable_collisions link1="${tf_prefix}wrist_2_link" link2="${tf_prefix}wrist_3_link" reason="Adjacent" />
   </xacro:macro>
 </robot>

File: ws_dependencies/description_beerpong/urdf/full_robot.urdf.xacro (robot description, xacro)
@@ -9,5 +9,5 @@
    <xacro:arg name="ur_type" default="ur5x"/>
    <!-- parameters -->
-   <xacro:arg name="prefix" default="ur_" />
+   <xacro:arg name="tf_prefix" default="ur_" />
    <xacro:arg name="joint_limit_params" default="$(find ur_description)/config/$(arg ur_type)/joint_limits.yaml"/>
    <xacro:arg name="kinematics_params" default="$(find ur_description)/config/$(arg ur_type)/default_kinematics.yaml"/>
@@ -54,5 +54,5 @@
    <xacro:ur_robot
      name="$(arg name)"
-     tf_prefix="$(arg prefix)"
+     tf_prefix="$(arg tf_prefix)"
      parent="world"
      joint_limits_parameters_file="$(arg joint_limit_params)"
@@ -108,5 +108,5 @@
       <plugin filename="libign_ros2_control-system.so" name="ign_ros2_control::IgnitionROS2ControlPlugin">
         <parameters>$(arg simulation_controllers)</parameters>
-        <controller_manager_node_name>$(arg prefix)controller_manager</controller_manager_node_name>
+        <controller_manager_node_name>$(arg tf_prefix)controller_manager</controller_manager_node_name>
       </plugin>
     </gazebo>
@@ -114,8 +114,8 @@
     <!--Greifer + Kamerahalter + Kamera Macro importieren -->
     <xacro:include filename="$(find description_beerpong)/urdf/gripper_macro.urdf.xacro"/>
-    <xacro:gripper_camera prefix="$(arg prefix)" parent="tool0" origin_xyz="0 0 0" origin_rpy="0 0 3.1415"/>
+    <xacro:gripper_camera tf_prefix="$(arg tf_prefix)" parent="$(arg tf_prefix)tool0" origin_xyz="0 0 0" origin_rpy="0 0 3.1415"/>
     <!--Neobotix Macro importieren -->
     <xacro:include filename="$(find neo_mpo_500-2)/robot_model/mpo_500_macro.urdf.xacro"/>
-    <xacro:neobotix parent="base_link" origin_xyz="0 -0.205 -0.805" origin_rpy="0 0 1.57075"/>
+    <xacro:neobotix parent="world" origin_xyz="0 -0.205 -0.805" origin_rpy="0 0 1.57075"/>
     <!--Neobotix cabin-->
     <joint name="neobotix_to_cabin" type="fixed">
@@ -136,5 +136,5 @@
           <mesh filename="package://description_beerpong/meshes/collision/cabin.dae" scale="0.001 0.001 0.001"/>
         </geometry>
-        <material name="$(arg prefix)red" />
+        <material name="$(arg tf_prefix)red" />
       </collision>
     </link>
@@ -151,5 +151,5 @@
           <mesh filename="package://description_beerpong/meshes/visual/becherspender.stl" scale="0.001 0.001 0.001"/>
         </geometry>
-        <material name="$(arg prefix)grey" />
+        <material name="$(arg tf_prefix)grey" />
       </visual>
       <collision>
@@ -158,5 +158,5 @@
           <mesh filename="package://description_beerpong/meshes/collision/becherspender.stl" scale="0.001 0.001 0.001"/>
         </geometry>
-        <material name="$(arg prefix)red" />
+        <material name="$(arg tf_prefix)red" />
       </collision>
     </link>
