Commit message: add prefix to ur

File: ws_dependencies/description_beerpong/urdf/gripper_macro.urdf.xacro (robot description, xacro)
@@ -4,13 +4,13 @@
   <xacro:include filename="$(find description_beerpong)/urdf/materials.urdf.xacro" />
 <!--build the gripper links and joints using a macro, which will be called in the diy_gripper_model.urdf.xacro while launching-->
-  <xacro:macro name="gripper_camera" params="prefix parent origin_xyz origin_rpy">
-    <xacro:materials prefix="${prefix}"/>
-    <joint name="${prefix}gripper_to_parent" type="fixed">
+  <xacro:macro name="gripper_camera" params="tf_prefix parent origin_xyz origin_rpy">
+    <xacro:materials tf_prefix="${tf_prefix}"/>
+    <joint name="${tf_prefix}gripper_to_parent" type="fixed">
         <parent link="${parent}"/>
-        <child link="${prefix}camera_mount_link"/>
+        <child link="${tf_prefix}camera_mount_link"/>
         <origin xyz="${origin_xyz}" rpy="${origin_rpy}"/>
     </joint>
 <!-- Camera Mount-->
-    <link name="${prefix}camera_mount_link">
+    <link name="${tf_prefix}camera_mount_link">
       <visual>
         <origin xyz="0 0 0" rpy="0 0 0" />
@@ -18,5 +18,5 @@
           <mesh filename="package://description_beerpong/meshes/visual/Kamera_Mount.stl" scale="0.001 0.001 0.001"/>
         </geometry>
-        <material name="${prefix}grey" />
+        <material name="${tf_prefix}grey" />
       </visual>
       <collision>
@@ -25,16 +25,16 @@
           <mesh filename="package://description_beerpong/meshes/collision/Kamera_Mount.stl" scale="0.001 0.001 0.001"/>
         </geometry>
-        <material name="${prefix}red" />
+        <material name="${tf_prefix}red" />
       </collision>
     </link>
 <!-- Gripper + Finger + Adapter-Plate-->
-    <joint name="${prefix}gripper_joint" type="fixed">
+    <joint name="${tf_prefix}gripper_joint" type="fixed">
     <!-- Position zueinander wird in den joints angepasst (nicht in links)-->
       <origin xyz="0 0 0.0245" rpy="1.57075 0 3.1415" />
-      <parent link="${prefix}camera_mount_link" />
-      <child link="${prefix}gripper_link" />
+      <parent link="${tf_prefix}camera_mount_link" />
+      <child link="${tf_prefix}gripper_link" />
       <axis xyz="0 0 1" />
     </joint>
-    <link name="${prefix}gripper_link">
+    <link name="${tf_prefix}gripper_link">
       <visual>
         <origin xyz="0 0 0" rpy="0 0 0" />
@@ -42,5 +42,5 @@
           <mesh filename="package://description_beerpong/meshes/visual/greifer_beerpong_baugruppe_aussen_greifen.stl" scale="0.001 0.001 0.001"/>
         </geometry>
-        <material name="${prefix}grey" />
+        <material name="${tf_prefix}grey" />
       </visual>
       <collision>
@@ -49,12 +49,12 @@
           <mesh filename="package://description_beerpong/meshes/collision/greifer_beerpong_baugruppe_aussen_greifen.stl" scale="0.001 0.001 0.001"/>
         </geometry>
-        <material name="${prefix}red" />
+        <material name="${tf_prefix}red" />
       </collision>
     </link>
 <!-- Realsense-Camera -->
-    <joint name="${prefix}camera_joint" type="fixed">
+    <joint name="${tf_prefix}camera_joint" type="fixed">
       <origin xyz="0 0.098 0.074" rpy="0 0 3.1415" />
-      <parent link="${prefix}camera_mount_link" />
-      <child link="${prefix}camera_link" />
+      <parent link="${tf_prefix}camera_mount_link" />
+      <child link="${tf_prefix}camera_link" />
       <axis xyz="0 0 1" />
     </joint>
@@ -66,5 +66,5 @@
       <origin xyz="0 0.098 0.074" rpy="0 0 0"/>
     </xacro:sensor_d415> -->
-    <link name="${prefix}camera_link">
+    <link name="${tf_prefix}camera_link">
       <visual>
         <origin xyz="0 0 0" rpy="0 0 0" />
@@ -72,5 +72,5 @@
           <mesh filename="package://description_beerpong/meshes/visual/realsense415.stl" scale="1 1 1"/>
         </geometry>
-        <material name="${prefix}grey" />
+        <material name="${tf_prefix}grey" />
       </visual>
       <collision>
@@ -79,8 +79,8 @@
           <mesh filename="package://description_beerpong/meshes/collision/realsense415.stl" scale="1 1 1"/>
         </geometry>
-        <material name="${prefix}red" />
+        <material name="${tf_prefix}red" />
       </collision>
     </link>
-    <!-- <link name="${prefix}camera_link">
+    <!-- <link name="${tf_prefix}camera_link">
       <visual>
         <origin xyz="0 0 0" rpy="0 0 0" />
@@ -88,5 +88,5 @@
           <mesh filename="package://description_beerpong/meshes/visual/realsense415.stl" scale="1 1 1"/>
         </geometry>
-        <material name="${prefix}grey" />
+        <material name="${tf_prefix}grey" />
       </visual>
       <collision>
@@ -95,14 +95,14 @@
           <mesh filename="package://description_beerpong/meshes/collision/realsense415.stl"  scale="1 1 1"/>
         </geometry>
-        <material name="${prefix}red" />
+        <material name="${tf_prefix}red" />
       </collision>
     </link> -->
     <!--add a TCP Link for convenience, show TCP reference set in rviz-->
-    <joint name="${prefix}tcp_joint" type="fixed">
+    <joint name="${tf_prefix}tcp_joint" type="fixed">
         <origin xyz="0 0.112 0" rpy="1.57075 0 3.1415"/>
-        <parent link="${prefix}gripper_link"/>
-        <child link="${prefix}tcp_link"/>
+        <parent link="${tf_prefix}gripper_link"/>
+        <child link="${tf_prefix}tcp_link"/>
     </joint>
-    <link name="${prefix}tcp_link"/>
+    <link name="${tf_prefix}tcp_link"/>
   </xacro:macro>
 </robot>

File: ws_dependencies/description_beerpong/urdf/materials.urdf.xacro (robot description, xacro)
@@ -5,30 +5,30 @@
 -->
 <robot xmlns:xacro="http://wiki.ros.org/xacro">
-  <xacro:macro name="materials" params="prefix">
-    <material name="${prefix}black">
+  <xacro:macro name="materials" params="tf_prefix">
+    <material name="${tf_prefix}black">
       <color rgba="0.0 0.0 0.0 1.0"/>
     </material>
-    <material name="${prefix}blue">
+    <material name="${tf_prefix}blue">
       <color rgba="0.0 0.0 0.8 1.0"/>
     </material>
-    <material name="${prefix}green">
+    <material name="${tf_prefix}green">
       <color rgba="0.0 0.8 0.0 1.0"/>
     </material>
-    <material name="${prefix}yellow">
+    <material name="${tf_prefix}yellow">
       <color rgba="1.0 1.0 0.0 1.0"/>
     </material>
-    <material name="${prefix}grey">
+    <material name="${tf_prefix}grey">
       <color rgba="0.6 0.6 0.6 1.0"/>
     </material>
-    <material name="${prefix}orange">
+    <material name="${tf_prefix}orange">
       <color rgba="${255/255} ${108/255} ${10/255} 1.0"/>
     </material>
-    <material name="${prefix}brown">
+    <material name="${tf_prefix}brown">
       <color rgba="${222/255} ${207/255} ${195/255} 1.0"/>
     </material>
-    <material name="${prefix}red">
+    <material name="${tf_prefix}red">
       <color rgba="0.8 0.0 0.0 1.0"/>
     </material>
-    <material name="${prefix}white">
+    <material name="${tf_prefix}white">
       <color rgba="1.0 1.0 1.0 1.0"/>
     </material>

Commit message: Camera link TF updated

File: ws_dependencies/beerpong_moveit_config/srdf/beerpong_macro.srdf.xacro (robot description, xacro)
@@ -68,5 +68,5 @@
     <disable_collisions link1="${tf_prefix}wrist_3_link" link2="${tf_prefix}camera_mount_link" reason="Adjacent" />
     <disable_collisions link1="${tf_prefix}camera_mount_link" link2="${tf_prefix}gripper_link" reason="Adjacent" />
-    <disable_collisions link1="${tf_prefix}camera_mount_link" link2="${tf_prefix}camera_link" reason="Never" />
+    <disable_collisions link1="${tf_prefix}camera_mount_link" link2="camera_link" reason="Never" />
     <!--disable cabin and cup_dispeser collisions-->
     <disable_collisions link1="cabin_link" link2="cup_dispenser_link" reason="Adjacent" />

File: ws_dependencies/description_beerpong/urdf/gripper_macro.urdf.xacro (robot description, xacro)
@@ -56,5 +56,5 @@
       <origin xyz="0 0.098 0.074" rpy="0 0 3.1415" />
       <parent link="${tf_prefix}camera_mount_link" />
-      <child link="${tf_prefix}camera_link" />
+      <child link="camera_link" />
       <axis xyz="0 0 1" />
     </joint>
@@ -66,5 +66,5 @@
       <origin xyz="0 0.098 0.074" rpy="0 0 0"/>
     </xacro:sensor_d415> -->
-    <link name="${tf_prefix}camera_link">
+    <link name="camera_link">
       <visual>
         <origin xyz="0 0 0" rpy="0 0 0" />

Commit message: added horizontal collision plane for ur robot

File: ws_dependencies/beerpong_moveit_config/srdf/beerpong_macro.srdf.xacro (robot description, xacro)
@@ -71,4 +71,8 @@
     <!--disable cabin and cup_dispeser collisions-->
     <disable_collisions link1="cabin_link" link2="cup_dispenser_link" reason="Adjacent" />
+    <!--disable collisions with collision plane-->
+    <disable_collisions link1="cabin_link" link2="collision_plane_link" reason="Adjacent" />
+    <disable_collisions link1="${tf_prefix}base_link" link2="collision_plane_link" reason="Adjacent" />
+    <disable_collisions link1="cup_dispenser_link" link2="collision_plane_link" reason="Adjacent" />
   </xacro:macro>
 </robot>

File: ws_dependencies/description_beerpong/urdf/full_robot.urdf.xacro (robot description, xacro)
@@ -161,3 +161,18 @@
       </collision>
     </link>
+    <!-- collision plane  (UR and collision plane are fixed at world link)-->
+    <joint name="ur_to_collision_plane" type="fixed">
+        <origin xyz="0.0 0.0 0.0" rpy="0.0 0.0 0.0" />
+        <parent link="world"/>
+        <child link="collision_plane_link"/>
+    </joint>
+    <link name="collision_plane_link">
+      <collision>
+        <origin xyz="0 0 -0.02" rpy="0 0 0" />
+        <geometry>
+          <cylinder radius="1.0" length="0.02"/>
+        </geometry>
+        <material name="$(arg tf_prefix)red" />
+      </collision>
+    </link>
 </robot>

Commit message: Setup URDF of UR without Neobotix and add visual for collision plate surface

File: ws_dependencies/beerpong_moveit_config/srdf/beerpong_macro.srdf.xacro (robot description, xacro)
@@ -45,5 +45,5 @@
     <!--DISABLE COLLISIONS - By default it is assumed that any link of the robot could potentially come into collision with any other link in the robot. This tag disables collision checking between a specified pair of links. -->
     <!--disable neobotix internal collisions-->
-    <disable_collisions link1="base_footprint" link2="mpo_500_wheel_front_left_link" reason="Adjacent" />
+    <!-- <disable_collisions link1="base_footprint" link2="mpo_500_wheel_front_left_link" reason="Adjacent" />
     <disable_collisions link1="base_footprint" link2="mpo_500_wheel_front_right_link" reason="Adjacent" />
     <disable_collisions link1="base_footprint" link2="mpo_500_wheel_back_left_link" reason="Adjacent" />
@@ -53,5 +53,5 @@
     <disable_collisions link1="base_footprint" link2="lidar_2_link" reason="Adjacent" />
     <disable_collisions link1="base_footprint" link2="cabin_link" reason="Adjacent" />
-    <disable_collisions link1="cabin_link" link2="${tf_prefix}base_link_inertia" reason="Adjacent" />
+    <disable_collisions link1="cabin_link" link2="${tf_prefix}base_link_inertia" reason="Adjacent" /> -->
     <disable_collisions link1="${tf_prefix}base_link" link2="${tf_prefix}base_link_inertia" reason="Adjacent" />
     <disable_collisions link1="${tf_prefix}base_link_inertia" link2="${tf_prefix}shoulder_link" reason="Adjacent" />
@@ -69,8 +69,8 @@
     <disable_collisions link1="${tf_prefix}camera_mount_link" link2="${tf_prefix}gripper_link" reason="Adjacent" />
     <disable_collisions link1="${tf_prefix}camera_mount_link" link2="camera_link" reason="Never" />
-    <!--disable cabin and cup_dispeser collisions-->
-    <disable_collisions link1="cabin_link" link2="cup_dispenser_link" reason="Adjacent" />
+    <!-- disable cabin and cup_dispeser collisions
+    <disable_collisions link1="cabin_link" link2="cup_dispenser_link" reason="Adjacent" /> -->
     <!--disable collisions with collision plane-->
-    <disable_collisions link1="cabin_link" link2="collision_plane_link" reason="Adjacent" />
+    <!-- <disable_collisions link1="cabin_link" link2="collision_plane_link" reason="Adjacent" /> -->
     <disable_collisions link1="${tf_prefix}base_link" link2="collision_plane_link" reason="Adjacent" />
     <disable_collisions link1="cup_dispenser_link" link2="collision_plane_link" reason="Adjacent" />

File: ws_dependencies/description_beerpong/urdf/full_robot.urdf.xacro (robot description, xacro)
@@ -116,8 +116,8 @@
     <xacro:gripper_camera tf_prefix="$(arg tf_prefix)" parent="$(arg tf_prefix)tool0" origin_xyz="0 0 0" origin_rpy="0 0 3.1415"/>
     <!--Neobotix Macro importieren -->
-    <xacro:include filename="$(find neo_mpo_500-2)/robot_model/mpo_500_macro.urdf.xacro"/>
-    <xacro:neobotix parent="world" origin_xyz="0 -0.205 -0.805" origin_rpy="0 0 1.57075"/>
+    <!-- <xacro:include filename="$(find neo_mpo_500-2)/robot_model/mpo_500_macro.urdf.xacro"/>
+    <xacro:neobotix parent="world" origin_xyz="0 -0.205 -0.805" origin_rpy="0 0 1.57075"/> -->
     <!--Neobotix cabin-->
-    <joint name="neobotix_to_cabin" type="fixed">
+    <!-- <joint name="neobotix_to_cabin" type="fixed">
         <origin xyz="0.072 0 0.386" rpy="0 0 -1.57075" />
         <parent link="base_link"/>
@@ -138,9 +138,10 @@
         <material name="$(arg tf_prefix)red" />
       </collision>
-    </link>
+    </link> -->
     <!--Cup dispenser-->
     <joint name="neobotix_to_cup_dispenser" type="fixed">
-        <origin xyz="-0.115 0.256 1.433" rpy="3.1415 0 3.1415" />
-        <parent link="base_link"/>
+        <!-- <origin xyz="-0.115 0.256 1.433" rpy="3.1415 0 3.1415" /> -->
+        <origin xyz="-0.256 -0.33 0.635" rpy="3.1415 0 -1.57075" />
+        <parent link="world"/>
         <child link="cup_dispenser_link"/>
     </joint>
@@ -175,4 +176,11 @@
         <material name="$(arg tf_prefix)red" />
       </collision>
+      <visual>
+        <origin xyz="0 0 -0.02" rpy="0 0 0" />
+        <geometry>
+          <cylinder radius="1.0" length="0.02"/>
+        </geometry>
+        <material name="$(arg tf_prefix)grey" />
+      </visual>
     </link>
 </robot>

Commit message: disable all collisions

File: ws_dependencies/beerpong_moveit_config/srdf/beerpong_macro.srdf.xacro (robot description, xacro)
@@ -25,5 +25,5 @@
       <joint name="${tf_prefix}wrist_3_joint" value="0" />
     </group_state>
-    <group_state name="${tf_prefix}up" group="${tf_prefix}${name}_manipulator">
+    <group_state name="${tf_prefix}up" group="${name}_manipulator">
       <joint name="${tf_prefix}elbow_joint" value="0" />
       <joint name="${tf_prefix}shoulder_lift_joint" value="-1.5707" />
@@ -33,5 +33,5 @@
       <joint name="${tf_prefix}wrist_3_joint" value="0" />
     </group_state>
-    <group_state name="${tf_prefix}test_configuration" group="${tf_prefix}${name}_manipulator">
+    <group_state name="${tf_prefix}test_configuration" group="${name}_manipulator">
       <joint name="${tf_prefix}elbow_joint" value="1.4" />
       <joint name="${tf_prefix}shoulder_lift_joint" value="-1.62" />
@@ -69,6 +69,6 @@
     <disable_collisions link1="${tf_prefix}camera_mount_link" link2="${tf_prefix}gripper_link" reason="Adjacent" />
     <disable_collisions link1="${tf_prefix}camera_mount_link" link2="camera_link" reason="Never" />
-    <!-- disable cabin and cup_dispeser collisions
-    <disable_collisions link1="cabin_link" link2="cup_dispenser_link" reason="Adjacent" /> -->
+    <!-- disable cabin and cup_dispeser collisions -->
+    <disable_collisions link1="cabin_link" link2="cup_dispenser_link" reason="Adjacent" />
     <!--disable collisions with collision plane-->
     <disable_collisions link1="cabin_link" link2="collision_plane_link" reason="Adjacent" />

File: ws_dependencies/neo_mpo_500-2-humble/robot_model/mpo_500_macro.urdf.xacro (robot description, xacro)
@@ -1,10 +1,10 @@
 <?xml version="1.0" encoding="utf-8"?>
 <robot xmlns:xacro="http://ros.org/wiki/xacro">
-  <xacro:macro name="neobotix" params="parent origin_xyz origin_rpy">
-      <joint name="neobotix_to_parent" type="fixed">
+  <xacro:macro name="neobotix"> <!-- params="parent origin_xyz origin_rpy" -->
+      <!-- <joint name="neobotix_to_parent" type="fixed">
           <parent link="${parent}"/>
           <child link="base_link"/>
           <origin xyz="${origin_xyz}" rpy="${origin_rpy}"/>
-      </joint>
+      </joint> -->
       <!-- Base Macro-->
       <link name="base_link"/>
